File: EMG_sensing_draft/EMG_sensing_draft.kicad_sch (KiCad schematic)
At the start: 63 parts, among them J1 EMG_SIGNAL, J2 USB_A_0480370001, J3 DEBUG, U1 W25Q128JV, U2 RN4871-I/RM140, U3 RP2040, U4 MCP1702T-3302E_CB, U5 NCS4325DR2G, U6 MCP6021, U7 MCP6N11-002E/SN, Y1 12MHz

Commit message: added level shifter and second order low pass filter
Parts:
- removed R19: 316, symbol Device:R
- added C16: .033uF, symbol Device:C
- added C18: .33uF, symbol Device:C
- added R15, R20: 909, symbol Device:R
- added R17: 9.09k, symbol Device:R
- added R21: 453, symbol Device:R
- C15: value 0.33uF -> .33uF
- R14: value 909 -> 453
- renumbered C16 to C17, C17 to C19, C18 to C20, C19 to C21, C20 to C22, R15 to R16, R16 to R18, R17 to R19, R18 to R22, R20 to R23, R21 to R24, R22 to R25, R23 to R26
Connections:
- net +1.65V: now also R14.1; no longer U5.5 (IN2+)
- net GND: now also C16.1, C18.2, R20.1
- net V_SIGNAL: now also C16.2, R17.2; no longer C15.2, R14.1, U5.7 (OUT2)
- net at C15.1, R14.2, U5.6 (IN2-): now also R15.1
- net at U5.8 (OUT3), U5.9 (IN3-): now also R21.2
- new net: C18.1, R20.2, R21.1, U5.5 (IN2+)
- new net: C15.2, R15.2, R17.1, U5.7 (OUT2)
Other:
- moved on the sheet: C12
