File: kicad/EMG_sensing_draft/EMG_sensing_draft.kicad_sch (KiCad schematic)
At the start: 161 parts, among them J1 USB_A_0480370001, J2 Conn_01x09, J3 DEBUG, U1 MCP6N11-002E/SN, U10 RP2040, U11 RN4871-I/RM140, U12 MCP1702T-3302E_CB, U13 Opamp_MCP6024T-E/ST, U14 Opamp_MCP6024T-E/ST, U15 Opamp_MCP6024T-E/ST, U16 MCP6021, U17 Opamp_MCP6024T-E/ST, U2 MCP6N11-002E/SN, U3 MCP6N11-002E/SN, U4 W25Q128JV, U5 MCP6N11-002E/SN, U6 ISL90462WIH627Z-TKCT-ND, U7 ISL90462WIH627Z-TKCT-ND, U8 ISL90462WIH627Z-TKCT-ND, U9 ISL90462WIH627Z-TKCT-ND, Y1 12MHz

Commit message: organized parts on layout
Parts:
- J2: footprint (none) -> Connector_PinSocket_2.54mm:PinSocket_1x09_P2.54mm_Vertical
Connections:
- net V_SIGNAL_ONE: now also C43.1, R59.2
- net V_SIGNAL_TWO: no longer C43.1, R59.2
Changed lines of the file:
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@@
   (junction (at 434.34 220.98) (diameter 0) (color 0 0 0 0)
   )
-  (junction (at 41.275 487.68) (diameter 0) (color 0 0 0 0)
-  )
   (junction (at 434.34 102.87) (diameter 0) (color 0 0 0 0)
   )
@@
   (junction (at 349.25 88.9) (diameter 0) (color 0 0 0 0)
   )
-  (junction (at 40.005 353.06) (diameter 0) (color 0 0 0 0)
-  )
   (junction (at 627.38 184.15) (diameter 0) (color 0 0 0 0)
   )
@@
   (junction (at 72.39 176.53) (diameter 0) (color 0 0 0 0)
   )
-  (junction (at 39.37 255.27) (diameter 0) (color 0 0 0 0)
-  )
   (junction (at 407.67 100.33) (diameter 0) (color 0 0 0 0)
   )
@@
   (junction (at 98.425 401.32) (diameter 0) (color 0 0 0 0)
   )
-  (junction (at 42.545 425.45) (diameter 0) (color 0 0 0 0)
-  )
   (junction (at 308.61 39.37) (diameter 0) (color 0 0 0 0)
   )
@@
     (effects (font (size 1.27 1.27)) (justify left bottom))
   )
-  (label "V_SIGNAL_TWO" (at 441.96 102.87 0)
+  (label "V_SIGNAL_ONE" (at 441.96 102.87 0)
     (effects (font (size 1.27 1.27)) (justify left bottom))
   )
@@
     (pin "1")
   )
-  (symbol (lib_id "power:PWR_FLAG") (at 41.275 487.68 0) (unit 1)
-    (in_bom yes) (on_board yes)
-    (property "Reference" "#FLG03" (id 0) (at 41.275 485.775 0)
-      (effects (font (size 1.27 1.27)) hide)
-    )
-    (property "Value" "PWR_FLAG" (id 1) (at 41.275 490.22 0))
-    (property "Footprint" "" (id 2) (at 41.275 487.68 0)
-      (effects (font (size 1.27 1.27)) hide)
-    )
-    (property "Datasheet" "~" (id 3) (at 41.275 487.68 0)
-      (effects (font (size 1.27 1.27)) hide)
-    )
-    (pin "1")
-  )
   (symbol (lib_id "Device:LED_Filled") (at 151.13 146.05 180) (unit 1)
     (in_bom yes) (on_board yes)
@@
     (pin "")
   )
-  (symbol (lib_id "power:PWR_FLAG") (at 40.005 353.06 0) (unit 1)
-    (in_bom yes) (on_board yes)
-    (property "Reference" "#FLG02" (id 0) (at 40.005 351.155 0)
-      (effects (font (size 1.27 1.27)) hide)
-    )
-    (property "Value" "PWR_FLAG" (id 1) (at 40.005 355.6 0))
-    (property "Footprint" "" (id 2) (at 40.005 353.06 0)
-      (effects (font (size 1.27 1.27)) hide)
-    )
-    (property "Datasheet" "~" (id 3) (at 40.005 353.06 0)
-      (effects (font (size 1.27 1.27)) hide)
-    )
-    (pin "1")
-  )
   (symbol (lib_id "Device:R") (at 402.59 111.76 90) (unit 1)
     (in_bom yes) (on_board yes)
@@
     (pin "")
   )
-  (symbol (lib_id "power:PWR_FLAG") (at 39.37 255.27 0) (unit 1)
-    (in_bom yes) (on_board yes)
-    (property "Reference" "#FLG01" (id 0) (at 39.37 253.365 0)
-      (effects (font (size 1.27 1.27)) hide)
-    )
-    (property "Value" "PWR_FLAG" (id 1) (at 39.37 257.81 0))
-    (property "Footprint" "" (id 2) (at 39.37 255.27 0)
-      (effects (font (size 1.27 1.27)) hide)
-    )
-    (property "Datasheet" "~" (id 3) (at 39.37 255.27 0)
-      (effects (font (size 1.27 1.27)) hide)
-    )
-    (pin "1")
-  )
   (symbol (lib_id "Connector_Generic:Conn_01x09") (at 341.63 50.8 0) (mirror y) (unit 1)
     (in_bom yes) (on_board yes) (fields_autoplaced)
     (property "Reference" "J2" (id 0) (at 341.63 34.29 0))
     (property "Value" "Conn_01x09" (id 1) (at 341.63 36.83 0))
-    (property "Footprint" "" (id 2) (at 341.63 50.8 0)
+    (property "Footprint" "Connector_PinSocket_2.54mm:PinSocket_1x09_P2.54mm_Vertical" (id 2) (at 341.63 50.8 0)
       (effects (font (size 1.27 1.27)) hide)
     )
@@
     (pin "2")
   )
-  (symbol (lib_id "power:PWR_FLAG") (at 42.545 425.45 0) (unit 1)
-    (in_bom yes) (on_board yes)
-    (property "Reference" "#FLG04" (id 0) (at 42.545 423.545 0)
-      (effects (font (size 1.27 1.27)) hide)
-    )
-    (property "Value" "PWR_FLAG" (id 1) (at 42.545 427.99 0))
-    (property "Footprint" "" (id 2) (at 42.545 425.45 0)
-      (effects (font (size 1.27 1.27)) hide)
-    )
-    (property "Datasheet" "~" (id 3) (at 42.545 425.45 0)
-      (effects (font (size 1.27 1.27)) hide)
-    )
-    (pin "1")
-  )
   (symbol (lib_id "power:GND") (at 19.05 359.41 0) (unit 1)
     (in_bom yes) (on_board yes) (fields_autoplaced)
@@
   )
   (symbol_instances
-    (path "/95677d46-12c9-48e8-9a53-689365fd8c1a"
-      (reference "#FLG01") (unit 1) (value "PWR_FLAG") (footprint "")
-    )
-    (path "/57d14188-020f-4fe7-b465-6d510fc8d66e"
-      (reference "#FLG02") (unit 1) (value "PWR_FLAG") (footprint "")
-    )
-    (path "/105b953c-6ef8-4366-9f17-5635cb51637e"
-      (reference "#FLG03") (unit 1) (value "PWR_FLAG") (footprint "")
-    )
-    (path "/97e6d676-456c-4bcb-883c-a272e0c77bf3"
-      (reference "#FLG04") (unit 1) (value "PWR_FLAG") (footprint "")
-    )
     (path "/ae2101c3-e8f2-4dc5-8a0d-3e77301d9500"
       (reference "#FLG05") (unit 1) (value "PWR_FLAG") (footprint "")
@@
     )
     (path "/9581e4b4-c1d5-4e6b-9f21-090634c92985"
-      (reference "J2") (unit 1) (value "Conn_01x09") (footprint "")
+      (reference "J2") (unit 1) (value "Conn_01x09") (footprint "Connector_PinSocket_2.54mm:PinSocket_1x09_P2.54mm_Vertical")
     )
     (path "/d0085297-953e-40bd-9507-9c0d496719e2"

Commit message: finished initial layout
Parts:
- removed C26, C27, C28, C46: 1uF, Capacitor_SMD:C_0603_1608Metric, symbol Device:C
- renumbered C29 to C26, C30 to C27, C31 to C28, C32 to C29, C33 to C30, C34 to C31, C35 to C32, C36 to C33, C37 to C34, C38 to C35, C39 to C36, C40 to C37, C41 to C38, C42 to C39, C43 to C40, C44 to C41, C45 to C42, C47 to C43, C48 to C44, C49 to C45, C50 to C46, C51 to C47
Connections:
- net DIF_AMP_FOUR_CAL: now also U10.11 (GPIO8); no longer U10.12 (GPIO9)
- net DIF_AMP_ONE_CAL: now also U10.18 (GPIO15); no longer U10.8 (GPIO6)
- net DIF_AMP_THREE_CAL: now also U10.14 (GPIO11); no longer U10.11 (GPIO8)
- net DIF_AMP_TWO_CAL: now also U10.17 (GPIO14); no longer U10.9 (GPIO7)
- net POT_CHANGE_FOUR: now also U10.8 (GPIO6); no longer U10.28 (GPIO17)
- net POT_CHANGE_ONE: now also U10.28 (GPIO17); no longer U10.14 (GPIO11)
- net POT_CHANGE_THREE: now also U10.12 (GPIO9); no longer U10.18 (GPIO15)
- net POT_CHANGE_TWO: now also U10.15 (GPIO12); no longer U10.16 (GPIO13)
- net POT_CS_FOUR: now also U10.9 (GPIO7); no longer U10.27 (GPIO16)
- net POT_CS_ONE: now also U10.27 (GPIO16); no longer U10.13 (GPIO10)
- net POT_CS_THREE: now also U10.13 (GPIO10); no longer U10.17 (GPIO14)
- net POT_CS_TWO: now also U10.16 (GPIO13); no longer U10.15 (GPIO12)

Commit message: finished four layer layout
Connections:
- net DIF_AMP_FOUR_CAL: now also U10.32 (GPIO21); no longer U10.11 (GPIO8)
- net DIF_AMP_THREE_CAL: now also U10.29 (GPIO18); no longer U10.14 (GPIO11)
- net POT_CHANGE_FOUR: now also U10.35 (GPIO23); no longer U10.8 (GPIO6)
- net POT_CHANGE_THREE: now also U10.31 (GPIO20); no longer U10.12 (GPIO9)
- net POT_CS_FOUR: now also U10.34 (GPIO22); no longer U10.9 (GPIO7)
- net POT_CS_THREE: now also U10.30 (GPIO19); no longer U10.13 (GPIO10)
- net at R9.1: now also U10.11 (GPIO8); no longer U10.34 (GPIO22)
- net at R10.1: now also U10.12 (GPIO9); no longer U10.35 (GPIO23)
- net at R11.1: now also U10.13 (GPIO10); no longer U10.36 (GPIO24)
- net at R12.1: now also U10.14 (GPIO11); no longer U10.37 (GPIO25)
Other:
- moved on the sheet: D1, D2, D3, D4, R10, R11, R12, R9

Commit message: wip
Connections:
- net DIF_AMP_FOUR_CAL: now also U10.35 (GPIO23); no longer U10.32 (GPIO21)
- net POT_CHANGE_FOUR: now also U10.37 (GPIO25); no longer U10.35 (GPIO23)
- net POT_CS_FOUR: now also U10.36 (GPIO24); no longer U10.34 (GPIO22)
Changed lines of the file:
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@@
   (junction (at 407.67 93.98) (diameter 0) (color 0 0 0 0)
   )
-  (no_connect (at 137.16 156.21))
   (no_connect (at 137.16 59.69))
   (no_connect (at 237.49 107.95))
@@
   (no_connect (at 186.69 92.71))
   (no_connect (at 237.49 90.17))
-  (no_connect (at 137.16 151.13))
+  (no_connect (at 137.16 140.97))
+  (no_connect (at 137.16 135.89))
   (no_connect (at 185.42 55.245))
   (no_connect (at 137.16 64.77))
@@
     (effects (font (size 1.27 1.27)) (justify left bottom))
   )
-  (label "POT_CHANGE_FOUR" (at 137.16 146.05 0)
+  (label "POT_CHANGE_FOUR" (at 137.16 156.21 0)
     (effects (font (size 1.27 1.27)) (justify left bottom))
   )
@@
     (effects (font (size 1.27 1.27)) (justify left bottom))
   )
-  (label "POT_CS_FOUR" (at 137.16 140.97 0)
+  (label "POT_CS_FOUR" (at 137.16 151.13 0)
     (effects (font (size 1.27 1.27)) (justify left bottom))
   )
@@
     (effects (font (size 1.27 1.27)) (justify left bottom))
   )
-  (label "DIF_AMP_FOUR_CAL" (at 137.16 135.89 0)
-    (effects (font (size 1.27 1.27)) (justify left bottom))
-  )
+  (label "DIF_AMP_FOUR_CAL" (at 137.16 146.05 0)
+    (effects (font (size 1.27 1.27)) (justify left bottom))
+  )

Commit message: Revert "Developed 4-Layer Layout for EMG Sensing Board"
Parts:
- removed C2, C3, C4: 1uF, Capacitor_SMD:C_0603_1608Metric, symbol Device:C
- removed C21, C22, C23, C27, C29, C43, C7, C8, C9: 0.1uF, Capacitor_SMD:C_0603_1608Metric, symbol Device:C
- removed C30, C31, C44: 10uF, Capacitor_SMD:C_0603_1608Metric, symbol Device:C
- removed C36, C37, C38, C39, C45, C46: .33uF, Capacitor_SMD:C_0603_1608Metric, symbol Device:C
- removed C41, C42, C47: .033uF, Capacitor_SMD:C_0603_1608Metric, symbol Device:C
- removed D10, D11, D12, D13, D14, D9: D, Diode_SMD:D_0805_2012Metric, symbol Device:D
- removed J2: Conn_01x09, Connector_PinSocket_2.54mm:PinSocket_1x09_P2.54mm_Vertical, symbol Connector_Generic:Conn_01x09
- removed R16, R17, R62: 787, Resistor_SMD:R_0603_1608Metric, symbol Device:R
- removed R21, R22, R63: 8.1k, Resistor_SMD:R_0603_1608Metric, symbol Device:R
- removed R24, R25, R27, R29, R30, R31, R42, R43, R45, R46, R64, R65, R66, R67, R68: 10k, Resistor_SMD:R_0603_1608Metric, symbol Device:R
- removed R35, R36, R37, R38, R39, R40, R6, R7, R8: 100k, Resistor_SMD:R_0603_1608Metric, symbol Device:R
- removed R49, R50, R51, R52, R69, R70: 453, Resistor_SMD:R_0603_1608Metric, symbol Device:R
- removed R55, R56, R57, R58, R71, R72: 909, Resistor_SMD:R_0603_1608Metric, symbol Device:R
- removed R60, R61, R73: 9.09k, Resistor_SMD:R_0603_1608Metric, symbol Device:R
- removed U14, U15, U17: Opamp_MCP6024T-E/ST, MCP6024:MCP6024T, symbol Device:Opamp_MCP6024T-E/ST
- removed U2, U3, U5: MCP6N11-002E/SN, MCP6N11:MCP6N11-002ESN, symbol MCP6N11:MCP6N11-002E/SN
- removed U7, U8, U9: ISL90462WIH627Z-TKCT-ND, ISL90462WIH627Z:ISL90462WIH627Z-TKCT-ND, symbol ISL90462WIH627Z-TKCT-ND:ISL90462WIH627Z-TKCT-ND
- added C26: 1uF, Capacitor_SMD:C_0603_1608Metric, symbol Device:C
- added J2: EMG_SIGNAL, Connector_PinHeader_2.54mm:PinHeader_1x03_P2.54mm_Vertical, symbol Connector_Generic:Conn_01x03
- renumbered C14 to C10, C15 to C11, C16 to C12, C17 to C13, C18 to C14, C19 to C15, C20 to C17, C24 to C22, C26 to C27, C32 to C29, C1 to C3, C33 to C30, C34 to C31, C35 to C32, C40 to C33, C5 to C4, C6 to C5, C10 to C6, C11 to C7, C12 to C8, C13 to C9, R12 to R10, R18 to R16, R19 to R17, R44 to R18, R20 to R19, R23 to R20, R26 to R21, R47 to R22, R48 to R23, R28 to R24, R32 to R25, R33 to R26, R34 to R27, R53 to R28, R54 to R29, R41 to R30, R59 to R31, R5 to R6, R9 to R7, R10 to R8, R11 to R9, U12 to U11, U16 to U14, U1 to U2, U4 to U3, U6 to U5, U10 to U6, U11 to U9
Connections:
- net +3.3V: now also C26.2
- net GND: now also C26.1
- net at R7.1: now also U6.34 (GPIO22); no longer U6.11 (GPIO8)
- net at U6.12 (GPIO9): no longer R8.1
- net at U6.13 (GPIO10): no longer R9.1
- net at U6.14 (GPIO11): no longer R10.1
- net DIF_AMP_CAL: now reaches U6.8 (GPIO6)
- net DIF_AMP_CAL: now also U2.8 (EN/*CAL)
- net POT_CS: now reaches U6.9 (GPIO7)
- net POT_CS: now also U5.4 (*CS)
- net Vout_1: now reaches R20.2, R21.1, R24.1, U13.13 (VINB-)
- net Vout_2_pos: now reaches D8.1 (K), R21.2, U13.10 (VINC+)
- net Vout_3: now reaches R18.2, R23.1, U13.8 (VOUTC)
- net Vout_2_neg: now reaches R18.1, R30.2, U13.9 (VINC-)
- net at R25.1: now also J2.1 (Pin_1)
- net at R26.1: now also J2.2 (Pin_2)
- net at R27.1: now also J2.3 (Pin_3)
- net DIF_AMP_FOUR_CAL: no longer names the net of U6.35 (GPIO23)
- net DIF_AMP_FOUR_CAL: now also R8.1
- net DIF_AMP_ONE_CAL: no longer names the net of U6.18 (GPIO15)
- net DIF_AMP_ONE_CAL: no longer U2.8 (EN/*CAL)
- net DIF_AMP_THREE_CAL: no longer names the net of U6.29 (GPIO18)
- net DIF_AMP_TWO_CAL: no longer names the net of U6.17 (GPIO14)
- net EMG_NODE_ONE renamed emg_node_one
- net emg_node_one: now also R26.2; no longer R25.2
- net EMG_NODE_THREE renamed emg_ref
- net EMG_NODE_TWO renamed emg_node_two
- net emg_node_two: now also R25.2; no longer R26.2
- net POT_CHANGE_FOUR: no longer names the net of U6.37 (GPIO25)
- net POT_CHANGE_FOUR: now also R10.1
- net POT_CHANGE_ONE: no longer names the net of U6.28 (GPIO17)
- net POT_CHANGE_ONE: no longer U5.3 (U/*D)
- net POT_CHANGE_THREE: no longer names the net of U6.31 (GPIO20)
- net POT_CHANGE_TWO: no longer names the net of U6.15 (GPIO12)
- net POT_CS_FOUR: no longer names the net of U6.36 (GPIO24)
- net POT_CS_FOUR: now also R9.1
- net POT_CS_ONE: no longer names the net of U6.27 (GPIO16)
- net POT_CS_ONE: no longer U5.4 (*CS)
- net POT_CS_THREE: no longer names the net of U6.30 (GPIO19)
- net POT_CS_TWO: no longer names the net of U6.16 (GPIO13)
- net V_DIFF_ONE renamed V_DIFF
- net V_SIGNAL_FOUR renamed V_SIGNAL
- net V_SIGNAL: now also C33.1, R31.2
- removed net V_SIGNAL_ONE: C33.1, R31.2, U6.38 (GPIO26/ADC0)
- net V_SIGNAL_THREE: no longer names the net of U6.40 (GPIO28/ADC2)
- net V_SIGNAL_TWO: no longer names the net of U6.39 (GPIO27/ADC1)
- new net POT_CHANGE: U5.3 (U/*D), U6.11 (GPIO8)
- no-connect marks 11 -> 23
Other:
- moved on the sheet: C27, C31, C32, C33, D1, D2, D3, D4, D7, D8, R10, R18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

Commit message: added three channels for emg sensing
Parts:
- removed J2: EMG_SIGNAL, Connector_PinHeader_2.54mm:PinHeader_1x03_P2.54mm_Vertical, symbol Connector_Generic:Conn_01x03
- added C? (x6): .33uF, Capacitor_SMD:C_0603_1608Metric, symbol Device:C
- added C? (x6): 1uF, Capacitor_SMD:C_0603_1608Metric, symbol Device:C
- added C? (x9): 0.1uF, Capacitor_SMD:C_0603_1608Metric, symbol Device:C
- added C? (x3): .033uF, Capacitor_SMD:C_0603_1608Metric, symbol Device:C
- added C? (x3): 10uF, Capacitor_SMD:C_0603_1608Metric, symbol Device:C
- added D? (x6): D, Diode_SMD:D_0805_2012Metric, symbol Device:D
- added J?: Conn_01x09, symbol Connector_Generic:Conn_01x09
- added R? (x15): 10k, Resistor_SMD:R_0603_1608Metric, symbol Device:R
- added R? (x9): 100k, Resistor_SMD:R_0603_1608Metric, symbol Device:R
- added R? (x6): 909, Resistor_SMD:R_0603_1608Metric, symbol Device:R
- added R? (x3): 9.09k, Resistor_SMD:R_0603_1608Metric, symbol Device:R
- added R? (x6): 453, Resistor_SMD:R_0603_1608Metric, symbol Device:R
- added R? (x3): 8.1k, Resistor_SMD:R_0603_1608Metric, symbol Device:R
- added R? (x3): 787, Resistor_SMD:R_0603_1608Metric, symbol Device:R
- added U? (x15): Opamp_MCP6024T-E/ST, MCP6024:MCP6024T, symbol Device:Opamp_MCP6024T-E/ST
- added U? (x3): ISL90462WIH627Z-TKCT-ND, ISL90462WIH627Z:ISL90462WIH627Z-TKCT-ND, symbol ISL90462WIH627Z-TKCT-ND:ISL90462WIH627Z-TKCT-ND
- added U? (x3): MCP6N11-002E/SN, MCP6N11:MCP6N11-002ESN, symbol MCP6N11:MCP6N11-002E/SN
Connections:
- net +1.65V: now also R?.1, R?.1, R?.1, U?.12 (VINB+), U?.12 (VINB+), U?.12 (VINB+), U?.3 (VINA+), U?.3 (VINA+), U?.3 (VINA+), U?.5 (RW), U?.5 (RW), U?.5 (RW), U?.5 (VREF), U?.5 (VREF), U?.5 (VREF)
- net +3.3V: now also C?.1, C?.1, C?.1, C?.1, C?.1, C?.1, C?.1, C?.1, C?.1, C?.2, C?.2, C?.2, C?.2, C?.2, C?.2, U?.1 (VDD), U?.1 (VDD), U?.1 (VDD), U?.4 (VDD), U?.4 (VDD), U?.4 (VDD), U?.7 (VDD), U?.7 (VDD), U?.7 (VDD)
- net GND: now also C?.1, C?.1, C?.1, C?.1, C?.1, C?.1, C?.1, C?.1, C?.1, C?.2, C?.2, C?.2, C?.2, C?.2, C?.2, C?.2, C?.2, C?.2, C?.2, C?.2, C?.2, R?.1, R?.1, R?.1, U?.11 (VSS), U?.11 (VSS), U?.11 (VSS), U?.2 (GND), U?.2 (GND), U?.2 (GND), U?.4 (VSS), U?.4 (VSS), U?.4 (VSS)
- net Vout_1: now also R?.1, R?.1, R?.1, R?.1, R?.1, R?.1, R?.2, R?.2, R?.2, U?.13 (VINB-), U?.13 (VINB-), U?.13 (VINB-)
- net Vout_2_neg: now also R?.1, R?.1, R?.1, R?.2, R?.2, R?.2, U?.9 (VINC-), U?.9 (VINC-), U?.9 (VINC-)
- net Vout_2_pos: now also D?.1 (K), D?.1 (K), D?.1 (K), R?.2, R?.2, R?.2, U?.10 (VINC+), U?.10 (VINC+), U?.10 (VINC+)
- net Vout_3: now also R?.1, R?.1, R?.1, R?.2, R?.2, R?.2, U?.8 (VOUTC), U?.8 (VOUTC), U?.8 (VOUTC)
- net DIF_AMP_FOUR_CAL: now reaches U6.12 (GPIO9)
- net DIF_AMP_FOUR_CAL: now also U?.8 (EN/*CAL)
- net POT_CS_ONE: now reaches U6.13 (GPIO10)
- net POT_CS_ONE: now also U5.4 (*CS)
- net POT_CHANGE_ONE: now reaches U6.14 (GPIO11)
- net POT_CHANGE_ONE: now also U5.3 (U/*D)
- net POT_CS_TWO: now reaches U6.15 (GPIO12)
- net POT_CS_TWO: now also U?.4 (*CS)
- net POT_CHANGE_TWO: now reaches U6.16 (GPIO13)
- net POT_CHANGE_TWO: now also U?.3 (U/*D)
- net POT_CS_THREE: now reaches U6.17 (GPIO14)
- net POT_CS_THREE: now also U?.4 (*CS)
- net POT_CHANGE_THREE: now reaches U6.18 (GPIO15)
- net POT_CHANGE_THREE: now also U?.3 (U/*D)
- net POT_CS_FOUR: now reaches U6.27 (GPIO16)
- net POT_CS_FOUR: now also U?.4 (*CS)
- net POT_CHANGE_FOUR: now reaches U6.28 (GPIO17)
- net POT_CHANGE_FOUR: now also U?.3 (U/*D)
- net V_SIGNAL_ONE: now reaches U6.38 (GPIO26/ADC0)
- net V_SIGNAL_ONE: now also C33.1, R31.2
- net V_SIGNAL_TWO: now reaches U6.39 (GPIO27/ADC1)
- net V_SIGNAL_TWO: now also C?.1, R?.2
- net V_SIGNAL_THREE: now reaches U6.40 (GPIO28/ADC2)
- net V_SIGNAL_THREE: now also C?.1, R?.2
- net at R25.1: now also J?.1 (Pin_1)
- net at R26.1: now also J?.2 (Pin_2)
- net at R27.1: now also J?.3 (Pin_3)
- net DIF_AMP_CAL renamed DIF_AMP_ONE_CAL
- net POT_CHANGE renamed DIF_AMP_THREE_CAL
- net DIF_AMP_THREE_CAL: now also U?.8 (EN/*CAL); no longer U5.3 (U/*D)
- net POT_CS renamed DIF_AMP_TWO_CAL
- net DIF_AMP_TWO_CAL: now also U?.8 (EN/*CAL); no longer U5.4 (*CS)
- net V_DIFF renamed V_DIFF_ONE
- removed net V_SIGNAL: C33.1, R31.2, U6.41 (GPIO29/ADC3)
- net emg_node_one renamed EMG_NODE_ONE
- net EMG_NODE_ONE: now also R25.2; no longer R26.2
- net emg_node_two renamed EMG_NODE_TWO
- net EMG_NODE_TWO: now also R26.2; no longer R25.2
- net emg_ref renamed EMG_NODE_THREE
- net EMG_NODE_THREE: now also U?.2 (VIM)
- new net: D?.1 (K), D?.2 (A), U?.14 (VOUTB) (x3)
- new net: D?.2 (A), R?.1, R?.2 (x3)
- new net: J?.8 (Pin_8), R?.1
- new net: C?.1, R?.1, R?.2, U?.6 (VIND-) (x3)
- new net: C?.2, R?.1, R?.2, U?.7 (VOUTD) (x3)
- new net: C?.2, R?.2, R?.2, U?.5 (VIND+) (x3)
- new net: R?.1, R?.2, U?.1 (VOUTA) (x3)
- new net: C?.2, R?.1, U?.2 (VINA-) (x3)
- new net: R?.2, U?.1 (VFG), U?.6 (RH) (x3)
- new net: J?.5 (Pin_5), R?.1
- new net: J?.7 (Pin_7), R?.1
- new net: C?.1, R?.2 (x3)
- new net: J?.4 (Pin_4), R?.1
- new net: J?.6 (Pin_6), R?.1
- new net: J?.9 (Pin_9), R?.1
- new net EMG_NODE_EIGHT: R?.2, U?.3 (VIP)
- new net EMG_NODE_FIVE: R?.2, U?.2 (VIM)
- new net EMG_NODE_FOUR: R?.2, U?.3 (VIP)
- new net EMG_NODE_SEVEN: R?.2, U?.2 (VIM)
- new net EMG_NODE_SIX: R?.2, U?.3 (VIP)
- new net EMG_REF: R?.2
- new net V_DIFF_FOUR: R?.1, R?.1, U?.6 (VOUT)
- new net V_DIFF_THREE: R?.1, R?.1, U?.6 (VOUT)
- new net V_DIFF_TWO: R?.1, R?.1, U?.6 (VOUT)
- new net V_SIGNAL_FOUR: C?.1, R?.2, U6.41 (GPIO29/ADC3)
- no-connect marks 23 -> 11
