File: kicad/EMG_sensing_draft/EMG_sensing_draft.kicad_sch (KiCad schematic)
At the start: 173 parts, among them J1 USB_A_0480370001, J3 DEBUG, U11 MCP1702T-3302E_CB, U13 Opamp_MCP6024T-E/ST, U14 MCP6021, U2 MCP6N11-002E/SN, U3 W25Q128JV, U5 ISL90462WIH627Z-TKCT-ND, U6 RP2040, U9 RN4871-I/RM140, Y1 12MHz

Commit message: cleaned up four channel schematic
Parts:
- removed C? (x6): .33uF, Capacitor_SMD:C_0603_1608Metric, symbol Device:C
- removed C? (x3): 1uF, Capacitor_SMD:C_0603_1608Metric, symbol Device:C
- removed C? (x3): .033uF, Capacitor_SMD:C_0603_1608Metric, symbol Device:C
- removed C? (x3): 10uF, Capacitor_SMD:C_0603_1608Metric, symbol Device:C
- removed C? (x3): 0.1uF, Capacitor_SMD:C_0603_1608Metric, symbol Device:C
- removed D? (x6): D, Diode_SMD:D_0805_2012Metric, symbol Device:D
- removed R? (x15): 10k, Resistor_SMD:R_0603_1608Metric, symbol Device:R
- removed R? (x6): 909, Resistor_SMD:R_0603_1608Metric, symbol Device:R
- removed R? (x3): 9.09k, Resistor_SMD:R_0603_1608Metric, symbol Device:R
- removed R? (x6): 453, Resistor_SMD:R_0603_1608Metric, symbol Device:R
- removed R? (x3): 8.1k, Resistor_SMD:R_0603_1608Metric, symbol Device:R
- removed R? (x3): 787, Resistor_SMD:R_0603_1608Metric, symbol Device:R
- removed U? (x15): Opamp_MCP6024T-E/ST, MCP6024:MCP6024T, symbol Device:Opamp_MCP6024T-E/ST
- added C27, C28, C46: 1uF, Capacitor_SMD:C_0603_1608Metric, symbol Device:C
- added C30, C32, C47: 0.1uF, Capacitor_SMD:C_0603_1608Metric, symbol Device:C
- added C33, C34, C48: 10uF, Capacitor_SMD:C_0603_1608Metric, symbol Device:C
- added C39, C40, C41, C42, C49, C50: .33uF, Capacitor_SMD:C_0603_1608Metric, symbol Device:C
- added C44, C45, C51: .033uF, Capacitor_SMD:C_0603_1608Metric, symbol Device:C
- added D10, D11, D12, D13, D14, D9: D, Diode_SMD:D_0805_2012Metric, symbol Device:D
- added R16, R17, R62: 787, Resistor_SMD:R_0603_1608Metric, symbol Device:R
- added R21, R22, R63: 8.1k, Resistor_SMD:R_0603_1608Metric, symbol Device:R
- added R24, R25, R27, R29, R30, R31, R42, R43, R45, R46, R64, R65, R66, R67, R68: 10k, Resistor_SMD:R_0603_1608Metric, symbol Device:R
- added R49, R50, R51, R52, R69, R70: 453, Resistor_SMD:R_0603_1608Metric, symbol Device:R
- added R55, R56, R57, R58, R71, R72: 909, Resistor_SMD:R_0603_1608Metric, symbol Device:R
- added R60, R61, R73: 9.09k, Resistor_SMD:R_0603_1608Metric, symbol Device:R
- added U14, U15, U17: Opamp_MCP6024T-E/ST, MCP6024:MCP6024T, symbol Device:Opamp_MCP6024T-E/ST
- gave numbers to parts that had none: 25
- renumbered C3 to C1, C6 to C10, C7 to C11, C8 to C12, C9 to C13, C10 to C14, C11 to C15, C12 to C16, C13 to C17, C14 to C18, C15 to C19, C17 to C20, C22 to C24, C27 to C29, C28 to C31, C29 to C35, C30 to C36, C31 to C37, C32 to C38, C33 to C43, C4 to C5, C5 to C6, R8 to R10, R9 to R11, R10 to R12, R16 to R18, R17 to R19, R19 to R20, R20 to R23, R21 to R26, R24 to R28, R25 to R32, R26 to R33, R27 to R34, R30 to R41, R18 to R44, R22 to R47, R23 to R48, R6 to R5, R28 to R53, R29 to R54, R31 to R59, R7 to R9, U2 to U1, U6 to U10, U9 to U11, U11 to U12, U14 to U16, U3 to U4, U5 to U6
Connections:
- net +1.65V: now also R49.1, R51.1, R69.1, U14.12 (VINB+), U14.3 (VINA+), U15.12 (VINB+), U15.3 (VINA+), U17.12 (VINB+), U17.3 (VINA+)
- net +3.3V: now also C27.2, C28.2, C30.2, C32.2, C46.2, C47.2, U14.4 (VDD), U15.4 (VDD), U17.4 (VDD)
- net GND: now also C27.1, C28.1, C30.1, C32.1, C40.1, C42.1, C44.2, C45.2, C46.1, C47.1, C50.1, C51.2, R56.1, R58.1, R72.1, U14.11 (VSS), U15.11 (VSS), U17.11 (VSS)
- net V_DIFF_FOUR: now also R62.1
- net V_DIFF_THREE: now also R16.1
- net V_DIFF_TWO: now also R17.1
- net V_SIGNAL_FOUR: now also C51.1, R73.2
- net V_SIGNAL_ONE: no longer C43.1, R59.2
- net V_SIGNAL_THREE: now also C44.1, R60.2
- net V_SIGNAL_TWO: now also C43.1, R59.2, C45.1, R61.2
- net Vout_1: no longer names the net of R23.2, R26.1, R28.1, U13.13 (VINB-)
- net Vout_2_neg: no longer names the net of R41.2, R44.1, U13.9 (VINC-)
- net Vout_2_pos: no longer names the net of D8.1 (K), R26.2, U13.10 (VINC+)
- net Vout_3: no longer names the net of R44.2, R48.1, U13.8 (VOUTC)
- new net: C40.2, R50.2, R56.2, U14.5 (VIND+)
- new net: C39.1, R49.2, R55.1, U14.6 (VIND-)
- new net: C39.2, R55.2, R60.1, U14.7 (VOUTD)
- new net: C48.1, R62.2
- new net: C48.2, R63.1, U17.2 (VINA-)
- new net: C42.2, R52.2, R58.2, U15.5 (VIND+)
- new net: C49.1, R69.2, R71.1, U17.6 (VIND-)
- new net: C49.2, R71.2, R73.1, U17.7 (VOUTD)
- new net: D10.1 (K), R27.2, U14.10 (VINC+)
- new net: R45.2, R50.1, U14.8 (VOUTC)
- new net: R42.2, R45.1, U14.9 (VINC-)
- new net: R21.2, R24.1, U14.1 (VOUTA)
- new net: C33.2, R21.1, U14.2 (VINA-)
- new net: R25.2, R29.1, R31.1, U15.13 (VINB-)
- new net: D12.1 (K), R29.2, U15.10 (VINC+)
- new net: D10.2 (A), D9.1 (K), U14.14 (VOUTB)
- new net: D11.1 (K), D12.2 (A), U15.14 (VOUTB)
- new net: D11.2 (A), R31.2, R43.1
- new net: C33.1, R16.2
- new net: C41.2, R57.2, R61.1, U15.7 (VOUTD)
- new net: C41.1, R51.2, R57.1, U15.6 (VIND-)
- new net: C50.2, R70.2, R72.2, U17.5 (VIND+)
- new net: R63.2, R64.1, U17.1 (VOUTA)
- new net: R22.2, R25.1, U15.1 (VOUTA)
- new net: C34.2, R22.1, U15.2 (VINA-)
- new net: R43.2, R46.1, U15.9 (VINC-)
- new net: D9.2 (A), R30.2, R42.1
- new net: R67.2, R68.1, U17.9 (VINC-)
- new net: R68.2, R70.1, U17.8 (VOUTC)
- new net: R24.2, R27.1, R30.1, U14.13 (VINB-)
- new net: R64.2, R65.1, R66.1, U17.13 (VINB-)
- new net: D13.2 (A), R66.2, R67.1
- new net: C34.1, R17.2
- new net: D14.1 (K), R65.2, U17.10 (VINC+)
- new net: D13.1 (K), D14.2 (A), U17.14 (VOUTB)
- new net: R46.2, R52.1, U15.8 (VOUTC)
Other:
- moved on the sheet: C26, C29, C37, C38, C43, D7, D8, R26, R28, R41, R44, R47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
