File: kicad/EMG_sensing_draft/EMG_sensing_draft.kicad_pcb (KiCad board)
At the start: 2 copper layers, 161 parts, among them J1 USB_A_0480370001, J2 Conn_01x09, J3 DEBUG, U1 MCP6N11-002E/SN, U10 RP2040, U11 RN4871-I/RM140, U12 MCP1702T-3302E_CB, U13 Opamp_MCP6024T-E/ST, U14 Opamp_MCP6024T-E/ST, U15 Opamp_MCP6024T-E/ST, U16 MCP6021, U17 Opamp_MCP6024T-E/ST, U2 MCP6N11-002E/SN, U3 MCP6N11-002E/SN, U4 W25Q128JV, U5 MCP6N11-002E/SN, U6 ISL90462WIH627Z-TKCT-ND, U7 ISL90462WIH627Z-TKCT-ND, U8 ISL90462WIH627Z-TKCT-ND, U9 ISL90462WIH627Z-TKCT-ND, Y1 12MHz

Commit message: placed filtering components
Parts:
- removed the C35 at (95.7, 78.7)
- moved C5 141.6 mm to (213.5, 65.1), turned to -90 degrees
- moved U4 132.2 mm to (210.0, 63.3), turned to -90 degrees
- moved R14 125.5 mm to (209.1, 98.6)
- moved D6 123.9 mm to (212.4, 98.6), turned to 180 degrees
- moved J1 123.6 mm to (211.4, 90.0), turned to 90 degrees
- moved R26 115.5 mm to (190.0, 65.8)
- moved U11 114.6 mm to (200.5, 56.0)
- moved C24 114.1 mm to (206.0, 93.2)
- moved U10 113.4 mm to (201.8, 68.8), turned to -90 degrees
- moved U12 112.9 mm to (206.0, 95.7)
- moved R18 112.4 mm to (202.4, 96.5), turned to 180 degrees
- moved R4 112.3 mm to (208.6, 74.6)
- moved C25 112.2 mm to (205.7, 98.3)
- moved U16 112.0 mm to (201.5, 94.0)
- moved R23 110.9 mm to (187.0, 67.3)
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- renumbered C36 to C35, C37 to C36, C38 to C37, C39 to C38, C40 to C39, C41 to C40, C42 to C41, C43 to C42, C44 to C43, C45 to C44, C46 to C45, C47 to C46, C48 to C47, C49 to C48, C50 to C49, C51 to C50
Connections:
- U10 pad 11: /DIF_AMP_THREE_CAL -> /POT_CHANGE_TWO
- U10 pad 12: /DIF_AMP_FOUR_CAL -> /POT_CS_ONE
- U10 pad 13: /POT_CS_ONE -> /POT_CHANGE_ONE
- U10 pad 14: /POT_CHANGE_ONE -> /DIF_AMP_ONE_CAL
- U10 pad 15: /POT_CS_TWO -> /DIF_AMP_THREE_CAL
- U10 pad 16: /POT_CHANGE_TWO -> /POT_CS_THREE
- U10 pad 17: /POT_CS_THREE -> /POT_CHANGE_THREE
- U10 pad 18: /POT_CHANGE_THREE -> /DIF_AMP_FOUR_CAL
- U10 pad 8: /DIF_AMP_ONE_CAL -> /DIF_AMP_TWO_CAL
- U10 pad 9: /DIF_AMP_TWO_CAL -> /POT_CS_TWO
Routing:
- net +3.3V: track 0.00 -> 118.8 mm
- net /V_SIGNAL_FOUR: track 0.00 -> 44.0 mm
- net /V_SIGNAL_THREE: track 0.00 -> 35.6 mm
- net /POT_CS_ONE: track 0.00 -> 30.8 mm
- net /POT_CHANGE_ONE: track 0.00 -> 26.7 mm
- net /DIF_AMP_ONE_CAL: track 0.00 -> 24.9 mm
- net /EMG_NODE_SEVEN: track 0.00 -> 21.9 mm
- net /USB_D-: track 0.00 -> 20.7 mm
- net /EMG_NODE_EIGHT: track 0.00 -> 20.5 mm
- net GND: track 0.00 -> 20.1 mm
- net Net-(R25-Pad2): track 0.00 -> 19.6 mm
- net Net-(D14-Pad1): track 0.00 -> 19.5 mm
- net /V_SIGNAL_TWO: track 0.00 -> 18.5 mm
- net /USB_D+: track 0.00 -> 18.2 mm
- net Net-(D10-Pad1): track 0.00 -> 17.8 mm
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- added copper zone on B.Cu, net GND
Other:
- board outline added: 72.4 x 62.6 mm

Commit message: started routing power lines
Parts:
- moved U8 0.12 mm to (169.7, 96.5)
Routing:
- net +1.65V: track 3.25 -> 67.0 mm, vias 0 -> 2
- net +3.3V: track 118.8 -> 131.3 mm
- net Net-(D14-Pad1): track 19.5 -> 17.3 mm
- net GND: track 20.1 -> 21.7 mm
- net /EMG_NODE_SEVEN: track 21.9 -> 22.7 mm
- net /EMG_NODE_EIGHT: track 20.5 -> 21.0 mm
