File: kicad/EMG_sensing_draft/EMG_sensing_draft.kicad_pcb (KiCad board)
At the start: 2 copper layers, 161 parts, among them J1 USB_A_0480370001, J2 Conn_01x09, J3 DEBUG, U1 MCP6N11-002E/SN, U10 RP2040, U11 RN4871-I/RM140, U12 MCP1702T-3302E_CB, U13 Opamp_MCP6024T-E/ST, U14 Opamp_MCP6024T-E/ST, U15 Opamp_MCP6024T-E/ST, U16 MCP6021, U17 Opamp_MCP6024T-E/ST, U2 MCP6N11-002E/SN, U3 MCP6N11-002E/SN, U4 W25Q128JV, U5 MCP6N11-002E/SN, U6 ISL90462WIH627Z-TKCT-ND, U7 ISL90462WIH627Z-TKCT-ND, U8 ISL90462WIH627Z-TKCT-ND, U9 ISL90462WIH627Z-TKCT-ND, Y1 12MHz

Commit message: finished initial layout
Parts:
- removed the C26 at (195.6, 157.5)
- removed the C27 at (160.0, 81.3)
- removed the C28 at (175.3, 50.8)
- removed the C46 at (175.3, 116.8)
- moved C5 203.6 mm to (268.7, 36.8)
- moved U4 193.7 mm to (267.2, 40.4)
- moved S2 190.6 mm to (267.4, 66.1), turned to 90 degrees
- moved R1 186.7 mm to (263.3, 74.5), turned to 90 degrees
- moved R2 179.0 mm to (263.3, 70.5), turned to -90 degrees
- moved S1 178.2 mm to (267.3, 74.2), turned to 90 degrees
- moved U11 177.2 mm to (258.8, 32.8), turned to -90 degrees
- moved R4 176.0 mm to (266.2, 47.5)
- moved R13 175.4 mm to (265.8, 81.4), turned to -90 degrees
- moved U10 175.0 mm to (259.5, 46.5), turned to -90 degrees
- moved R26 172.1 mm to (244.2, 36.5)
- moved R3 172.0 mm to (266.2, 49.1), turned to 180 degrees
- moved R14 171.4 mm to (263.7, 81.4), turned to -90 degrees
- moved D5 171.4 mm to (265.8, 84.6), turned to 90 degrees
- moved R12 170.6 mm to (261.6, 81.4), turned to -90 degrees
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- renumbered C29 to C26, C30 to C27, C31 to C28, C32 to C29, C33 to C30, C34 to C31, C35 to C32, C36 to C33, C37 to C34, C38 to C35, C39 to C36, C40 to C37, C41 to C38, C42 to C39, C43 to C40, C44 to C41, C45 to C42, C47 to C43, C48 to C44, C49 to C45, C50 to C46, C51 to C47
Connections:
- U10 pad 11: /DIF_AMP_THREE_CAL -> /DIF_AMP_FOUR_CAL
- U10 pad 12: /DIF_AMP_FOUR_CAL -> /POT_CHANGE_THREE
- U10 pad 13: /POT_CS_ONE -> /POT_CS_THREE
- U10 pad 14: /POT_CHANGE_ONE -> /DIF_AMP_THREE_CAL
- U10 pad 15: /POT_CS_TWO -> /POT_CHANGE_TWO
- U10 pad 16: /POT_CHANGE_TWO -> /POT_CS_TWO
- U10 pad 17: /POT_CS_THREE -> /DIF_AMP_TWO_CAL
- U10 pad 18: /POT_CHANGE_THREE -> /DIF_AMP_ONE_CAL
- U10 pad 27: /POT_CS_FOUR -> /POT_CS_ONE
- U10 pad 28: /POT_CHANGE_FOUR -> /POT_CHANGE_ONE
- U10 pad 8: /DIF_AMP_ONE_CAL -> /POT_CHANGE_FOUR
- U10 pad 9: /DIF_AMP_TWO_CAL -> /POT_CS_FOUR
Routing:
- net GND: track 0.00 -> 449.8 mm, vias 0 -> 44
- net +3.3V: track 0.00 -> 357.7 mm
- net +1.65V: track 0.00 -> 253.1 mm, vias 0 -> 2
- net /POT_CHANGE_FOUR: track 0.00 -> 98.3 mm, vias 0 -> 2
- net /DIF_AMP_FOUR_CAL: track 0.00 -> 96.3 mm, vias 0 -> 2
- net /POT_CS_FOUR: track 0.00 -> 95.0 mm, vias 0 -> 2
- net /POT_CHANGE_THREE: track 0.00 -> 94.3 mm, vias 0 -> 4
- net /POT_CS_THREE: track 0.00 -> 87.1 mm, vias 0 -> 4
- net Net-(R13-Pad1): track 0.00 -> 76.6 mm, vias 0 -> 2
- net /DIF_AMP_THREE_CAL: track 0.00 -> 76.0 mm, vias 0 -> 2
- net /DIF_AMP_TWO_CAL: track 0.00 -> 71.4 mm, vias 0 -> 4
- net /POT_CHANGE_TWO: track 0.00 -> 66.3 mm, vias 0 -> 2
- net /POT_CS_TWO: track 0.00 -> 61.8 mm, vias 0 -> 4
- net Net-(R2-Pad1): track 0.00 -> 61.6 mm, vias 0 -> 2
- net /USB_D+: track 0.00 -> 49.6 mm
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- added copper zone on B.Cu, net GND
Other:
- board outline added: 49.4 x 60.1 mm
